File: hardware/board/usb_isolated/usb_isolated.kicad_pcb (KiCad board)
At the start: 4 copper layers, 80 x 50 mm, 191 parts, among them J2 Conn_01x03_Male, J3 Conn_Triaxial, J4 AudioJack3, J5 USB_C_Receptacle_USB2.0, J6 Barrel_Jack_Switch, J7 Conn_Coaxial, SW2 SW_DIP_x02, U1 74LVCH2T45DC, U10 ADA4891-2, U11 LM27762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

Commit message: update usb isolated pcba layout
Parts:
- removed C11, C22, C23: 10uF, Capacitor_SMD:C_0805_2012Metric
- removed C16, C20, C21, C26, C28, C29, C38, C59, C60, C61, C62, C63, C64, C65, C69, C70, C71: 100nF, Capacitor_SMD:C_0402_1005Metric
- removed C24, C25: 100nF, Capacitor_SMD:C_0603_1608Metric
- removed C27, C41: 1uF, Capacitor_SMD:C_0402_1005Metric
- removed C30, C31, C68, C72: 160pF, Capacitor_SMD:C_0402_1005Metric
- removed C32, C35, C36, C57, C58: 1nF, Capacitor_SMD:C_0402_1005Metric
- removed C33, C34: 120pF, Capacitor_SMD:C_0402_1005Metric
- removed C40: 22uF, Capacitor_SMD:C_0805_2012Metric
- removed C42: 4.7uF, Capacitor_SMD:C_0603_1608Metric
- removed C43, C44, C50, C51: 2.2uF, Capacitor_SMD:C_0402_1005Metric
- removed C52: 300pF, Capacitor_SMD:C_0402_1005Metric
- removed C73, C74: 130pF, Capacitor_SMD:C_0402_1005Metric
- removed G1, G2: LOGO, LOGO
- removed H1: MountingHole_Pad, kicad_component_library:Terminal_Keystone_779x_EdgeMount_Horizontal
- removed J3: Conn_Triaxial, kicad_component_library:TRB_Trompeter_CBBJR79A_Horizontal
- removed R14: 100K, Resistor_SMD:R_1206_3216Metric
- removed R15: 100, Resistor_SMD:R_0402_1005Metric_Pad0.72x0.64mm_HandSolder
- removed R16, R17, R25, R45, R60, R61, R8: 4K7, Resistor_SMD:R_0402_1005Metric
- removed R18, R23: 127K, Resistor_SMD:R_0402_1005Metric
- removed R19: 976, Resistor_SMD:R_0402_1005Metric
- removed R20: 97K6, Resistor_SMD:R_0402_1005Metric
- removed R21, R22, R55, R66, R71: 100K, Resistor_SMD:R_0402_1005Metric
- removed R24: 1K05, Resistor_SMD:R_0402_1005Metric
- removed R26: 102K, Resistor_SMD:R_0402_1005Metric
- removed R27: 10K0, Resistor_SMD:R_0402_1005Metric
- removed R28, R29, R44: 49.9, Resistor_SMD:R_0402_1005Metric
- removed R32: 54K9, Resistor_SMD:R_0402_1005Metric
- removed R33: 53K6, Resistor_SMD:R_0402_1005Metric
- removed R34, R35: 51K, Resistor_SMD:R_0402_1005Metric
- removed R42, R43: 127, Resistor_SMD:R_0402_1005Metric
- removed R46: 133, Resistor_SMD:R_0402_1005Metric
- removed R47: 113, Resistor_SMD:R_0402_1005Metric
- removed R48, R72: 8K87, Resistor_SMD:R_0402_1005Metric
- removed R49, R51, R52, R53, R54, R56, R62, R63, R70, R74, R75: 1K00, Resistor_SMD:R_0402_1005Metric
- removed R50: 2K2, Resistor_SMD:R_0402_1005Metric
- removed R57, R58: 10K, Resistor_SMD:R_0402_1005Metric
- removed R59: 0, Resistor_SMD:R_0402_1005Metric_Pad0.72x0.64mm_HandSolder
- removed R64: 133K, Resistor_SMD:R_0402_1005Metric
- removed R65: 1K02, Resistor_SMD:R_0402_1005Metric
- removed R67: 10K2, Resistor_SMD:R_0402_1005Metric
- removed R68: 137, Resistor_SMD:R_0402_1005Metric
- removed R69: 121K, Resistor_SMD:R_0402_1005Metric
- removed R73: 115, Resistor_SMD:R_0402_1005Metric
- removed SW2: SW_DIP_x02, Button_Switch_SMD:SW_DIP_SPSTx02_Slide_9.78x7.26mm_W8.61mm_P2.54mm
- removed TP1: TestPoint, TestPoint:TestPoint_THTPad_D3.0mm_Drill1.5mm
- removed U10: ADA4891-2, Package_SO:MSOP-8_3x3mm_P0.65mm
- removed U11: LM27762, Package_SON:WSON-12-1EP_3x2mm_P0.5mm_EP1x2.65_ThermalVias
- removed U13: ADS7049, Package_SO:VSSOP-8_2.3x2mm_P0.5mm
- removed U14, U18: MAX4564EKA, Package_TO_SOT_SMD:SOT-23-8
- removed U17: ADA4891-1, Package_TO_SOT_SMD:SOT-23-5
- removed U6: ADA4891-4, Package_SO:TSSOP-14_4.4x5mm_P0.65mm
- removed U7: LTC6268xS8-10, Package_SO:SO-8_3.9x4.9mm_P1.27mm
- removed U8: REF2025, Package_TO_SOT_SMD:SOT-23-5
- removed U9: TS5A9411DCKR, Package_TO_SOT_SMD:SOT-363_SC-70-6
Routing:
- net GND: track 120.8 -> 56.4 mm, vias 313 -> 47
- net -2V5: track 55.6 -> 0.00 mm, vias 10 -> 0
- net /Lick Detection Analog Front End/triax_inner_shield: track 42.0 -> 0.00 mm, vias 20 -> 0
- net +2V5: track 27.7 -> 0.00 mm, vias 9 -> 0
- net GAIN_SEL_2V5: track 25.3 -> 0.00 mm, vias 2 -> 0
- net VREF_1V25: track 23.1 -> 0.00 mm, vias 2 -> 0
- net /100KHz Sine Wave/VSINE: track 22.7 -> 0.00 mm
- net /Harp Core RP2040 + Isolated USB/GAIN_SEL_DIP: track 22.1 -> 0.00 mm, vias 2 -> 0
- net /Harp Core RP2040 + Isolated USB/FREQ_SEL_DIP: track 19.6 -> 0.00 mm, vias 4 -> 0
- net Net-(R43-Pad2): track 17.2 -> 0.00 mm, vias 1 -> 0
- net Net-(U7--): track 16.1 -> 0.00 mm
- net Net-(R49-Pad1): track 14.7 -> 0.00 mm
- net +5V: track 27.2 -> 13.2 mm, vias 10 -> 5
- net GAIN_SEL: track 12.2 -> 0.00 mm
- net FREQ_SEL_2V5: track 12.2 -> 0.00 mm, vias 2 -> 0
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- removed copper zone on In2.Cu, net +2V5
- removed copper zone on In2.Cu, net -2V5
- removed copper zone on In1.Cu, net /Lick Detection Analog Front End/triax_inner_shield
Other:
- board text added: "Name Here"
- board text added: "QR Code Here"
- board text added: "SIPE Version, MMM DD, 20xx"
- board text removed: "(TTL) Lick Detected ↘"
- board text removed: "100KHz ←"
- board text removed: "125KHz →"
- board text removed: "Ground Lug (M4)"
- board text removed: "Lickety Split Lick Detector"
- board text removed: "Notes: • DIP switches control excitation signal amplitude and frequency. These settings are applied upon power-up, but they can be overwritten from the software (Harp) interface afterwards. • When using the 0.02Vpp excitation signal, the animal must share a ground with this board through the ground lug or barrel jack power plug. • When using 2 lick detectors with lick tubes spaced closely togethe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"
- board text removed: "Sonya Vasquez"
- board text removed: "Sub-millisecond, ephys-compatible rodent lick detection system."
- board text removed: "v0.8.0, May 17, 2024"
- board text removed: "← 0.02Vpp"
- board text removed: "↑ Lick Tube Input (Triax)"
- board text removed: "→ 2Vpp"
- board text removed: "↖ Filtered Detection Signal"
